File: MotherForSmoothie_preliminary.brd (EAGLE design)
At the start: 100 x 80 mm, 154 parts, among them IC14 TC4427, IC3 74AHC1G07DBV, J1 22-27-2031-03, J2 22-27-2041-04, J3 22-27-2041-04, J4 22-27-2031-03, J5 22-27-2041-04, J6 22-27-2041-04, M1 DRV8825, M10 DRV8825, M6 DRV8825, M7 DRV8825, Q1 IRF9530, Q12 ZXMN4A06, Q3 MOSFET-PCHANNELSMD, Q6 AOT240L, Q8 ZXMN4A06, U1 USD-SOCKETNEW, X11 MC2-G, X2 MC2-G, X3 USB-MICROB, X4 MC2-G, X6 MC2-G, X7 5566-20, X9 MC2-G

Commit message: Updated board and schematic
Parts:
- removed R9: 2k2, rcl:R0603
- added C9: .1uF, rcl:C0603
- added LED9: (no value), led:CHIPLED_0805
- added R16, R17: (no value), rcl:R0603
- C10: value .1uF -> 100n
- C8: value (none) -> 100n
- Q1: value IRF9530 -> SUP90P06-09L
- R1: value 2k2 -> ?
- moved R53 0.64 mm to (84.5, 70.5)
- turned LED1 to 270 degrees
Connections:
- removed net AGND: C11.C, C12.C, C5.C, C7.C, JP21.1, JP21.3, JP21.5, JP21.7
- removed net FLOW: C8.1, D2.A, D3.C, J4.3, R1.1, R9.1
- removed net N$29: JP4.2, LED1.A
- removed net VCC: IC3.5
- new net N$234234: JP4.1, LED1.C, R2.1
- new net N$39: IC3.4, R16.2
- new net N$41: LED9.A, R17.1
- net 3.3V: now also X7.11
- net GND: now also C11.C, C12.C, C5.C, C7.C, C9.1, JP21.1, JP21.3, JP21.5, JP21.7, LED9.C, RJ2.G+, RJ2.G-, RJ2.Y+, RJ2.Y-
- net N$34: now also C9.2, IC3.5
- net P1_22: now also C8.1, D2.A, D3.C, J4.3, R1.1
- net PLAY_LED: now also JP4.2, LED1.A; no longer JP4.1, LED1.C, R2.1
- net RESET: now also R16.1
- net VUSB: now also R17.2
Routing:
- net FLOW: track 95.1 -> 0.00 mm, vias 2 -> 0
- net P1_22: track 78.7 -> 173.7 mm, vias 4 -> 6
- net GND: track 722.5 -> 763.1 mm, vias 28 -> 35
- net AGND: track 29.8 -> 0.00 mm, vias 4 -> 0
- net MS0: track 140.8 -> 114.8 mm, vias 1 -> 3
- net N$34: track 3.01 -> 23.9 mm, vias 0 -> 1
- net N$39: track 0.00 -> 10.4 mm, vias 0 -> 2
- net N$234234: track 0.00 -> 8.23 mm, vias 0 -> 1
- net N$41: track 0.00 -> 5.67 mm, vias 0 -> 1
- net RESET: track 27.7 -> 33.0 mm, vias 2 -> 3
- net N$29: track 4.03 -> 0.00 mm
- net EN5: track 67.7 -> 63.8 mm
- net VUSB: track 0.00 -> 3.61 mm
- net N$15: track 100.2 -> 96.9 mm
- net EN4: track 47.9 -> 45.3 mm
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- added copper zone on layer 16, net VBB
Other:
- board text added: "bot"
- board text added: "top"

Commit message: More cleanup and fixes
Parts:
- removed C48, C61: 10uF, SparkFun:EIA3216
- removed C60: 100uF, rcl:E5-8,5
- removed D4: 15v, diode:SMB
- removed JP17, JP18, JP19: (no value), pinhead (3):1X04SMD
- removed JP20: JUMPER-3PTH, SparkFun:1X03
- removed JP30: (no value), pinhead (3):1X05SMD
- removed JP33: (no value), SparkFun:1X02
- removed LED5, LED6, LED7, LED8: (no value), led:CHIP-LED0805
- removed M10: DRV8825, selfmade2:DRV8825
- removed Q6: AOT240L, transistor-power:TO220BV
- removed Q8: ZXMN4A06, ipc-7351-transistor:SOT230P700X160-4N
- removed R57, R61, R62, R66: 10K, rcl:R0603
- removed R67: 1.5K, rcl:R0603
- removed R69, R70, R72, R78: 1k, rcl:R0603
- removed R71, R73, R75, R77, R79: 5k6, rcl:R0603
- removed S4: (no value), SparkFun:TACTILE_SWITCH_SMD
- added ATX, PLAY: (no value), led:CHIPLED_0805
- added AVCC: M01PTH, SparkFun:1X01
- added BIG, SMALL: (no value), led:CHIP-LED0805
- added C13, C14: 18pF, rcl:C0603
- added C25: 100uF, rcl:E5-8,5
- added D1: 1N4148, diode:MINIMELF
- added M2: DRV8825, selfmade2:DRV8825
- added MS1, MS2, MS3: (no value), pinhead (3):1X02SMD
- added PS_ON: (no value), jumper:JP1
- added Q2: MOSFET-PCHANNELSMD, SparkFun:SOT23-3
- added Q5: SUP90P06-09L, transistor-power:TO220BV
- added R31, R32, R38, R47, R48, R50: 10K, rcl:R0603
- added R33, R35, R37: 1k, rcl:R0603
- added R46: ?, rcl:R0603
- added R51: 5.6K, rcl:R0603
- added R52: 22R, rcl:R0603
- added R54: 2.2K, rcl:R0603
- added R55: 10k, rcl:R0603
- added RESET: (no value), SparkFun:TACTILE_SWITCH_SMD
- added XMAX, XMIN, YMAX, YMIN, ZMAX, ZMIN: (no value), SparkFun:1X03_NO_SILK
- C1, C2, C3: value 100uF -> 10uF; device rcl:E5-8,5 -> SparkFun:EIA3216
- C10: value 100n -> 100uF; device rcl:C0603 -> rcl:E5-8,5
- C11: value 10uF -> .1uF; device SparkFun:EIA3216 -> rcl:C0603
- C12, C21: value 10uF -> 100uF; device SparkFun:EIA3216 -> rcl:E5-8,5
- C22: value 18pF -> 100n
- C23: value 18pF -> 10uF; device rcl:C0603 -> SparkFun:EIA3216
- C24: value .1uF -> 100n
- C26: value 1uF -> 100uF; device rcl:C0603 -> rcl:E5-8,5
- C4, C9: value .1uF -> 10uF; device rcl:C0603 -> SparkFun:EIA3216
- C6: value 100uF -> .1uF; device rcl:E5-8,5 -> rcl:C0603
- C7: value 10uF -> 1uF; device SparkFun:EIA3216 -> rcl:C0603
- C8: value 100n -> .1uF
- D3: value 1N4148 -> 15v; device diode:MINIMELF -> diode:SMB
- J1: value 22-27-2031-03 -> 22-27-2041-04; device con-molex:6410-03 -> con-molex:6410-04
- J2: value 22-27-2041-04 -> 22-27-2031-03; device con-molex:6410-04 -> con-molex:6410-03
- JP1, JP4: value (none) -> FIDUCIAL1X2; device pinhead (3):1X02SMD -> SparkFun:FIDUCIAL-1X2
- JP10, JP8: value JUMPER-3PTH -> (none); device SparkFun:1X03 -> pinhead (3):1X05SMD
- JP11: value JUMPER-3PTH -> (none); device SparkFun:1X03 -> pinhead (3):1X06SMD
- JP12: device pinhead (3):1X02SMD -> pinhead (3):1X04SMD
- JP13: device pinhead (3):1X02SMD -> SparkFun:1X03_NO_SILK
- JP14: device pinhead (3):1X05SMD -> SparkFun:1X02
- JP15: device pinhead (3):1X03SMD -> pinhead (3):1X02SMD
- JP16: device jumper:JP1 -> pinhead (3):1X04SMD
- JP2: value (none) -> FIDUCIAL1X2; device pinhead (3):1X06SMD -> SparkFun:FIDUCIAL-1X2
- JP3: value JUMPER-3PTH -> FIDUCIAL1X2; device SparkFun:1X03 -> SparkFun:FIDUCIAL-1X2
- JP5: device pinhead (3):1X04SMD -> pinhead (3):1X03SMD
- JP6: value JUMPER-3PTH -> (none); device SparkFun:1X03 -> SparkFun:1X03_NO_SILK
- JP7, JP9: value JUMPER-3PTH -> (none); device SparkFun:1X03 -> pinhead (3):1X04SMD
- LED1, LED4: device led:CHIPLED_0805 -> led:CHIP-LED0805
- Q1: value SUP90P06-09L -> ZXMN4A06; device transistor-power:TO220BV -> ipc-7351-transistor:SOT230P700X160-4N
- Q3: value MOSFET-PCHANNELSMD -> AOT240L; device SparkFun:SOT23-3 -> transistor-power:TO220BV
- R1: value ? -> (none)
- R10: value 22R -> 10K; device resistor:R0603 -> rcl:R0603
- R11, R30: value 10k -> 10K; device resistor:R0603 -> rcl:R0603
- R12: value 5.6K -> 10K; device resistor:R0603 -> rcl:R0603
- R13: value 22R -> 5.6K
- R14: value 10k -> 22R
- R15: value 5.6K -> 10k
- R16: value (none) -> 10k; device rcl:R0603 -> resistor:R0603
- R17: value (none) -> 1.5K
- R18, R4: value 10K -> (none)
- R19, R24, R26, R27: value 10K -> 1k
- R2: value 1k -> 5.6K; device rcl:R0603 -> resistor:R0603
- R25, R28: value 2.2k -> 5k6
- R3: value (none) -> 1k
- R36: value 22R -> 5k6
- R39: value 2.2K -> 10K
- R41, R42: value 1k -> 2.2k
- R43: value 10k -> 5k6
- R45: value 10K -> 5k6
- R49: value 5.6K -> 10K
- R6: value 10K -> 22R; device rcl:R0603 -> resistor:R0603
- R7: value 10K -> 10k; device rcl:R0603 -> resistor:R0603
- R8: value 1k -> 10K
- X2: value MC2-G -> 5566-20; device con-phoenix-381_l:MC2-G -> con-molex:5566-20
- X3: value USB-MICROB -> MC2-G; device SparkFun:USB-MICROB -> con-phoenix-381_l:MC2-G
- X6: value MC2-G -> USB-MICROB; device con-phoenix-381_l:MC2-G -> SparkFun:USB-MICROB
- X7: value 5566-20 -> MC2-G; device con-molex:5566-20 -> con-phoenix-381_l:MC2-G
- moved JP4 113.8 mm to (1.27, 78.7), flipped to the bottom, turned to 0 degrees
- moved JP3 106.8 mm to (1.27, 78.7)
- moved X7 92.7 mm to (95.2, 74.3), turned to 90 degrees
- moved R53 89.9 mm to (17.8, 10.2)
- moved R26 86.5 mm to (98.4, 54.0), turned to 270 degrees
- moved JP1 85.5 mm to (98.4, 1.27), flipped to the bottom
- moved J1 80.5 mm to (57.1, 74.3), turned to 0 degrees
- moved C10 80.1 mm to (80.6, 8.89), flipped to the top, turned to 45 degrees
- moved JP7 79.1 mm to (17.8, 17.8)
- moved S1 78.6 mm to (92.1, 66.7), turned to 180 degrees
- moved C2 74.8 mm to (53.3, 17.8), flipped to the bottom, turned to 180 degrees
- moved X4 72.8 mm to (83.2, 2.54), turned to 0 degrees
- moved JP13 70.0 mm to (92.7, 23.5)
- moved R4 69.1 mm to (73.0, 22.2)
- moved X3 68.4 mm to (64.1, 2.54), flipped to the top, turned to 0 degrees
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- renumbered C27 to C15, C28 to C16, C29 to C17, C30 to C18, C34 to C19, C35 to C20, IC14 to IC2, IC3 to IC1, JP21 to THERM., JP34 to LEDS, LED14 to VBB, LED16 to FAN, LED9 to USB, LPC2 to LPC1, M6 to M4, M7 to M3, Q12 to Q4, R65 to R9, R68 to R22, R74 to R34, R76 to R40, R90 to R23, RJ2 to RJ1, SJ6 to SJ1, X11 to X5, X9 to X1
Connections:
- net +12V: now also C11.2, C23.A, J4.2, R51.1, X2.10; no longer C4.2, C48.A, J1.2, R49.1, X7.10
- net +5V: now also J2.1, X2.19, X2.20, X2.4, X2.6; no longer J4.1, X7.19, X7.20, X7.4, X7.6
- net 3.3V: now also C7.2, C8.2, C9.A, D1.C, JP11.6, JP12.1, JP13.1, JP7.1, JP9.1, MS1.2, MS2.2, MS3.2, Q2.2, R10.2, R11.2, R12.2, R30.2, R31.2, R32.2, R33.2, R38.2, R39.2, R46.2, R47.2, R48.2, R49.2, R50.2, R8.2, X2.1, X2.11, X2.2; no longer C21.A, C24.2, C26.2, D2.C, JP1.2, JP12.2, JP13.2, JP17.1, JP18.1, JP2.6, JP3.1, JP5.1, Q3.2, R1.2, R18.2, R19.2, R2.2, R24.2, R26.2, R27.2, R4.2, R45.2, R57.2, R6.2, R61.2, R62.2, R66.2, R7.2, X7.1, X7.11, X7.2
- net 5V: now also JP13.3, JP7.3; no longer JP17.3, JP3.3
- net AVCC: now also AVCC.1
- net DIR3: now also JP16.3; no longer JP19.3
- net DIR4: now also M2.16; no longer M1.16
- net DIR5: now also M1.16; no longer M10.16
- net EN3: now also JP16.1; no longer JP19.1
- net EN4: now also M2.9; no longer M1.9
- net EN5: now also M1.9; no longer M10.9
- net GND: now also ATX.C, C1.C, C10.-, C11.1, C12.-, C13.1, C14.1, C2.C, C21.-, C22.2, C23.C, C25.-, C26.-, C3.C, C4.C, C6.1, C7.1, C8.1, C9.C, D2.A, J2.2, JP10.5, JP11.1, JP12.2, JP14.2, JP16.4, JP5.1, JP8.5, LED1.C, LED2.C, LED3.C, M2.1, M2.7, PS_ON.2, Q1.3, Q3.S, R15.1, R16.1, R55.2, R7.2, RESET.3, RESET.4, X2.13, X2.15, X2.16, X2.17, X2.3, X2.5, X2.7, X4.2, X6.GND, X7.1, XMAX.2, XMIN.2, YMAX.2, YMIN.2, ZMAX.2, ZMIN.2; no longer C1.-, C10.1, C11.C, C12.C, C2.-, C21.C, C22.1, C23.1, C26.1, C3.-, C4.1, C48.C, C6.-, C60.-, C61.C, C7.C, C8.2, C9.1, D3.A, J4.2, JP10.2, JP11.2, JP14.5, JP15.1, JP16.2, JP17.2, JP18.2, JP19.4, JP2.1, JP30.5, JP33.2, JP5.2, JP6.2, JP8.2, LED5.C, LED6.C, LED7.C, LED8.C, M10.1, M10.7, Q6.S, Q8.3, R11.1, R14.2, R30.1, R43.2, S4.3, S4.4, X2.2, X3.GND, X4.1, X7.13, X7.15, X7.16, X7.17, X7.3, X7.5, X7.7
- net ISP_BOOT: now also R31.1, S1.1, S1.2; no longer R24.1, S2.1, S2.2
- net LED1: now also R26.2; no longer R29.2
- net LED2: now also R29.2; no longer R41.2
- net LED3: now also R35.2; no longer R42.2
- net LED4: now also R37.2; no longer R44.2
- net MISO1: now also JP11.3; no longer JP2.3
- net MOSFET_DRIVE: now also C10.+, R13.1, X4.1; no longer C60.+, R12.1, X2.1
- net MOSI1: now also JP11.2; no longer JP2.2
- net MS0: now also M2.10, MS3.1; no longer JP13.1, M10.10
- net MS1: now also M2.11, MS2.1; no longer JP12.1, M10.11
- net MS2: now also M2.12, MS1.1; no longer JP1.1, M10.12
- net N$1: now also X6.D+; no longer X3.D+
- net N$10: now also LED1.A, R26.1; no longer LED5.A, R29.1
- net N$105: now also BIG.A, R13.2; no longer LED2.A, R12.2
- net N$107: now also R52.1; no longer R36.1
- net N$11: now also J3.3, M2.5; no longer J6.3, M1.5
- net N$12: now also Q2.3, R17.2; no longer Q3.3, R67.2
- net N$126: now also R54.1; no longer R39.1
- net N$128: now also R51.2; no longer R49.2
- net N$13: now also J3.4, M2.6; no longer J6.4, M1.6
- net N$135: now also D3.A, Q5.G, R55.1; no longer D4.A, Q1.G, R53.1
- net N$14: now also JP13.2, R19.2, R24.2, R27.2, R44.2, XMAX.3, XMIN.3, YMAX.3, YMIN.3, ZMAX.3, ZMIN.3; no longer JP10.3, JP11.3, JP3.2, JP6.3, JP7.3, JP8.3, JP9.3, R69.2, R70.2, R72.2, R78.2
- net N$140: now also C24.2; no longer C10.2
- net N$146: now also J1.3, M1.5; no longer J5.3, M10.5
- net N$147: now also J1.4, M1.6; no longer J5.4, M10.6
- net N$148: now also J1.2, M1.4; no longer J5.2, M10.4
- net N$149: now also J1.1, M1.3; no longer J5.1, M10.3
- net N$15: now also R43.1, ZMIN.1; no longer JP6.1, R77.1
- net N$152: now also M1.14, R11.1; no longer M10.14, R57.1
- net N$153: now also M1.13, R12.1; no longer M10.13, R62.1
- net N$16: now also R19.1, XMIN.1; no longer JP11.1, R69.1
- net N$17: now also R49.1; no longer R4.1
- net N$18: now also R24.1, R25.1, XMAX.1; no longer JP10.1, R70.1, R71.1
- net N$19: now also R27.1, R28.1, YMIN.1; no longer JP9.1, R72.1, R73.1
- net N$2: now also X6.D-; no longer X3.D-
- net N$20: now also R36.1, YMAX.1; no longer JP8.1, R75.1
- net N$21: now also J3.2, M2.4; no longer J6.2, M1.4
- net N$22: now also J5.3; no longer J3.3
- net N$23: now also JP7.4; no longer JP17.4
- net N$234234: now also JP15.1, PLAY.C, R33.1; no longer JP4.1, LED1.C, R2.1
- net N$24: now also R44.1, R45.1, ZMAX.1; no longer JP7.1, R78.1, R79.1
- net N$25: now also J5.4; no longer J3.4
- net N$26: now also J5.2; no longer J3.2
- net N$27: now also R41.2, R42.2; no longer R25.2, R28.2
- net N$28: now also J5.1; no longer J3.1
- net N$3: now also J6.3; no longer J2.3
- net N$30: now also R47.1; no longer R18.1
- net N$31: now also J3.1, M2.3; no longer J6.1, M1.3
- net N$32: now also M2.14, R38.1; no longer M1.14, R6.1
- net N$33: now also M2.13, R39.1; no longer M1.13, R7.1
- net N$34: now also C6.2, R3.2, X2.9; no longer C9.2, R8.2, X7.9
- net N$35: now also X2.8; no longer X7.8
- net N$36: now also ATX.A, R3.1; no longer LED4.A, R8.1
- net N$37: now also PS_ON.1, X2.14; no longer JP16.1, X7.14
- net N$38: now also JP5.2, R4.1; no longer JP15.2, R3.1
- net N$39: now also R1.2; no longer R16.2
- net N$4: now also J6.4; no longer J2.4
- net N$40: now also R14.1; no longer R10.1
- net N$41: now also R18.1; no longer R17.1
- net N$5: now also LED4.A, R37.1; no longer LED8.A, R44.1
- net N$6: now also LED3.A, R35.1; no longer LED7.A, R42.1
- net N$67: now also R50.1; no longer R26.1
- net N$68: now also R48.1; no longer R27.1
- net N$7: now also LED2.A, R29.1; no longer LED6.A, R41.1
- net N$74: now also Q1.1, R6.1; no longer Q8.1, R13.1
- net N$8: now also J6.2; no longer J2.2
- net N$81: now also R2.2, SMALL.A; no longer LED3.A, R15.2
- net N$88: now also Q1.4, SMALL.C, X3.2; no longer LED3.C, Q8.4, X6.2
- net N$9: now also J6.1; no longer J2.1
- net N$92: now also BIG.C, Q3.D; no longer LED2.C, Q6.D
- net N$96: now also J4.1; no longer J1.1
- net P1_22: now also C22.1, D1.A, D2.C, J2.3, JP10.1, R46.1; no longer C8.1, D2.A, D3.C, J4.3, JP14.1, R1.1
- net P1_23: now also JP10.2; no longer JP14.2
- net P1_30: now also JP10.4; no longer JP14.4
- net P1_31: now also JP10.3; no longer JP14.3
- net P2.6: now also JP8.1, R52.2, R53.1; no longer JP30.1, R36.2, R43.1
- net P2.7: now also JP8.4; no longer JP30.4
- net P2.9: now also Q2.1; no longer Q3.1
- net PLAY: now also JP14.1, R32.1, S2.1, S2.2; no longer JP33.1, R45.1, S4.1, S4.2
- net PLAY_LED: now also JP15.2, PLAY.A; no longer JP4.2, LED1.A
- net POT_SCL: now also JP9.4; no longer JP18.4
- net POT_SDA: now also JP9.3; no longer JP18.3
- net PWM0: now also JP8.2, R6.2, R7.1; no longer JP30.2, R13.2, R14.1
- net PWM1: now also JP8.3, R16.2; no longer JP30.3, R11.2
- net PWM1_FET: now also Q3.G, R14.2; no longer Q6.G, R10.2
- net RESET: now also R1.1, R30.1, RESET.1, RESET.2; no longer R16.1, R19.1, S1.1, S1.2
- net RX_0: now also R4.2; no longer R3.2
- net SCK1: now also JP11.4; no longer JP2.4
- net SCL: now also JP12.4, R41.1; no longer JP5.4, R25.1
- net SDA: now also JP12.3, R42.1; no longer JP5.3, R28.1
- net SD_CD: now also JP6.3; no longer JP20.3
- net SD_CS: now also R8.1; no longer R66.1
- net SD_IRQ: now also JP6.1; no longer JP20.1
- net SD_MOSI: now also R10.1; no longer R61.1
- net SD_WP: now also JP6.2; no longer JP20.2
- net SMALL_MOSFET_POWER: now also C1.A, R2.1, X3.1; no longer C61.A, R15.1, X6.1
- net SSDFGSDFG: now also R15.2; no longer R30.2
- net SSEL1: now also JP11.5; no longer JP2.5
- net STP3: now also JP16.2; no longer JP19.2
- net STP4: now also M2.15; no longer M1.15
- net STP5: now also M1.15; no longer M10.15
- net TH1: now also C2.A; no longer C5.A
- net TH2: now also C3.A; no longer C7.A
- net TH3: now also C4.A; no longer C11.A
- net TH4: now also C5.A; no longer C12.A
- net TX_0: now also JP5.3; no longer JP15.3
- net USB_D+: now also C14.2, R17.1; no longer C23.2, R67.1
- net USB_D-: now also C13.2; no longer C22.2
- net VBB: now also C12.+, C21.+, C25.+, C26.+, D3.C, M2.8, Q5.S, R54.2; no longer C1.+, C2.+, C3.+, C6.+, D4.C, M10.8, Q1.S, R39.2
- net VBB_IN: now also Q5.D, X7.2; no longer Q1.D, X4.2
- net VUSB: now also R18.2, X6.VBUS; no longer R17.2, X3.VBUS
- net X_MAX: now also R25.2; no longer R71.2
- net Y_MAX: now also R36.2; no longer R75.2
- net Y_MIN: now also R28.2; no longer R73.2
- net Z_MAX: now also R45.2; no longer R79.2
- net Z_MIN: now also R43.2; no longer R77.2
Routing:
- net 3.3V: track 422.6 -> 417.2 mm
- net STP1: track 50.7 -> 47.9 mm
- net SSDFGSDFG: track 43.3 -> 41.2 mm
- net 5V: track 135.4 -> 133.3 mm
- net N$14: track 64.2 -> 62.4 mm
- net RESET: track 33.0 -> 31.2 mm
- net N$15: track 96.9 -> 95.2 mm
- net PLAY_LED: track 34.0 -> 32.3 mm
- net Y_MAX: track 18.0 -> 16.4 mm
- net ISP_BOOT: track 41.2 -> 39.5 mm
- net TD+: track 34.2 -> 32.8 mm
- net SDA: track 18.5 -> 17.1 mm
- net LED3: track 27.8 -> 26.3 mm
- net N$24: track 98.5 -> 97.1 mm
- net TH2: track 30.9 -> 29.6 mm
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Other:
- board text added: "+"
- board text added: "-"
- board text added: "3V3"
- board text added: "5V"
- board text added: "GND"
- board text removed: "1"
- board text removed: "2"
- board text removed: "3"
- board text removed: "4"
- board text removed: "PWM0"
- board text removed: "PWM1"
