File: MotherForSmoothie_preliminary.sch (EAGLE design)
At the start: 154 parts, among them IC14 TC4427, IC3 74AHC1G07DBV, J1 22-27-2031-03, J2 22-27-2041-04, J3 22-27-2041-04, J4 22-27-2031-03, J5 22-27-2041-04, J6 22-27-2041-04, M1 DRV8825, M10 DRV8825, M6 DRV8825, M7 DRV8825, Q1 IRF9530, Q12 ZXMN4A06, Q3 MOSFET-PCHANNELSMD, Q6 AOT240L, Q8 ZXMN4A06, U1 USD-SOCKETNEW, X11 MC2-G, X2 MC2-G, X3 USB-MICROB, X4 MC2-G, X6 MC2-G, X7 5566-20, X9 MC2-G

Commit message: Updated board and schematic
Parts:
- removed R9: 2k2, rcl:R-EU_R0603
- added C9: .1uF, rcl:C-EUC0603
- added LED9: (no value), led:LEDCHIPLED_0805
- added R16, R17: (no value), rcl:R-EU_R0603
- C10: value .1uF -> 100n
- C8: value (none) -> 100n
- Q1: value IRF9530 -> SUP90P06-09L
- R1: value 2k2 -> ?
Connections:
- removed net AGND: C11.-, C12.-, C5.-, C7.-, JP21.1, JP21.3, JP21.5, JP21.7
- removed net FLOW: C8.1, D2.A, D3.C, J4-3.S, R1.1, R9.1
- removed net N$29: JP4.2, LED1.A
- new net N$234234: JP4.1, LED1.C, R2.1
- new net N$39: IC3A.O, R16.2
- new net N$41: LED9.A, R17.1
- net 3.3V: now also X7-11.S
- net GND: now also C11.-, C12.-, C5.-, C7.-, C9.1, JP21.1, JP21.3, JP21.5, JP21.7, LED9.C, RJ2.G+, RJ2.G-, RJ2.Y+, RJ2.Y-
- net N$34: now also C9.2, IC3P.VCC
- net P1_22: now also C8.1, D2.A, D3.C, J4-3.S, R1.1
- net PLAY_LED: now also JP4.2, LED1.A; no longer JP4.1, LED1.C, R2.1
- net RESET: now also R16.1
- net VUSB: now also R17.2
Other:
- note added: "!!!"
- note added: "ATX psu connector"
- note added: "Ethernet Jack"
- note added: "FAN Mosfet"
- note added: "Flowmeter"
- note added: "Reverse Polarity Protection VBB"
- note removed: "16 th"
- note removed: "4th"
- note removed: "FULL"
- note removed: "GPIO Channel"
- note removed: "H"
- note removed: "HALF"
- note removed: "L"
- note removed: "MS1"
- note removed: "MS2"
- note removed: "SW002:"
- note removed: "Steckerbelegung pruefen"
- moved on the sheet: C2, C22, C4, C8, D2, D3, D4, FB1, H1, H2, H3, H4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

Commit message: More cleanup and fixes
Parts:
- removed C48, C61: 10uF, SparkFun:CAP_POL1206
- removed C60: 100uF, rcl:CPOL-EUE5-8.5
- removed D4: 15v, diode:ZENER-DIODESMB
- removed JP17, JP18, JP19: (no value), pinhead (3):PINHD-1X4_2.54-SMD
- removed JP20: JUMPER-3PTH, SparkFun:JUMPER-3PTH
- removed JP30: (no value), pinhead (3):PINHD-1X5_2.54-SMD
- removed JP33: (no value), SparkFun:M02PTH
- removed LED5, LED6, LED7, LED8: (no value), led:LEDCHIP-LED0805
- removed M10: DRV8825, selfmade2:DRV8825
- removed Q6: AOT240L, transistor-power:IRF540
- removed Q8: ZXMN4A06, ipc-7351-transistor:MOSFET-NCH_SOT-223
- removed R57, R61, R62, R66: 10K, rcl:R-EU_R0603
- removed R67: 1.5K, rcl:R-EU_R0603
- removed R69, R70, R72, R78: 1k, rcl:R-EU_R0603
- removed R71, R73, R75, R77, R79: 5k6, rcl:R-EU_R0603
- removed S4: (no value), SparkFun:TAC_SWITCHSMD
- added ATX, PLAY: (no value), led:LEDCHIPLED_0805
- added AVCC: M01PTH, SparkFun:M01PTH
- added BIG, SMALL: (no value), led:LEDCHIP-LED0805
- added C13, C14: 18pF, rcl:C-EUC0603
- added C25: 100uF, rcl:CPOL-EUE5-8.5
- added D1: 1N4148, diode:DIODE-MINIMELF
- added M2: DRV8825, selfmade2:DRV8825
- added MS1, MS2, MS3: (no value), pinhead (3):PINHD-1X2_2.54-SMD
- added PS_ON: (no value), jumper:JP1E
- added Q2: MOSFET-PCHANNELSMD, SparkFun:MOSFET-PCHANNELSMD
- added Q5: SUP90P06-09L, transistor-power:IRF9530
- added R31, R32, R38, R47, R48, R50: 10K, rcl:R-EU_R0603
- added R33, R35, R37: 1k, rcl:R-EU_R0603
- added R46: ?, rcl:R-EU_R0603
- added R51: 5.6K, rcl:R-EU_R0603
- added R52: 22R, rcl:R-EU_R0603
- added R54: 2.2K, rcl:R-EU_R0603
- added R55: 10k, rcl:R-EU_R0603
- added RESET: (no value), SparkFun:TAC_SWITCHSMD
- added XMAX, XMIN, YMAX, YMIN, ZMAX, ZMIN: (no value), SparkFun:M031X03_NO_SILK
- C1, C2, C3: value 100uF -> 10uF; device rcl:CPOL-EUE5-8.5 -> SparkFun:CAP_POL1206
- C10: value 100n -> 100uF; device rcl:C-EUC0603 -> rcl:CPOL-EUE5-8.5
- C11: value 10uF -> .1uF; device SparkFun:CAP_POL1206 -> rcl:C-EUC0603
- C12, C21: value 10uF -> 100uF; device SparkFun:CAP_POL1206 -> rcl:CPOL-EUE5-8.5
- C22: value 18pF -> 100n
- C23: value 18pF -> 10uF; device rcl:C-EUC0603 -> SparkFun:CAP_POL1206
- C24: value .1uF -> 100n
- C26: value 1uF -> 100uF; device rcl:C-EUC0603 -> rcl:CPOL-EUE5-8.5
- C4, C9: value .1uF -> 10uF; device rcl:C-EUC0603 -> SparkFun:CAP_POL1206
- C6: value 100uF -> .1uF; device rcl:CPOL-EUE5-8.5 -> rcl:C-EUC0603
- C7: value 10uF -> 1uF; device SparkFun:CAP_POL1206 -> rcl:C-EUC0603
- C8: value 100n -> .1uF
- D3: value 1N4148 -> 15v; device diode:DIODE-MINIMELF -> diode:ZENER-DIODESMB
- J1: value 22-27-2031-03 -> 22-27-2041-04; device con-molex:22-27-2031-03 -> con-molex:22-27-2041-04
- J2: value 22-27-2041-04 -> 22-27-2031-03; device con-molex:22-27-2041-04 -> con-molex:22-27-2031-03
- JP1, JP4: value (none) -> FIDUCIAL1X2; device pinhead (3):PINHD-1X2_2.54-SMD -> SparkFun:FIDUCIAL1X2
- JP10, JP8: value JUMPER-3PTH -> (none); device SparkFun:JUMPER-3PTH -> pinhead (3):PINHD-1X5_2.54-SMD
- JP11: value JUMPER-3PTH -> (none); device SparkFun:JUMPER-3PTH -> pinhead (3):PINHD-1X6_2.54-SMD
- JP12: device pinhead (3):PINHD-1X2_2.54-SMD -> pinhead (3):PINHD-1X4_2.54-SMD
- JP13: device pinhead (3):PINHD-1X2_2.54-SMD -> SparkFun:M031X03_NO_SILK
- JP14: device pinhead (3):PINHD-1X5_2.54-SMD -> SparkFun:M02PTH
- JP15: device pinhead (3):PINHD-1X3_2.54-SMD -> pinhead (3):PINHD-1X2_2.54-SMD
- JP16: device jumper:JP1E -> pinhead (3):PINHD-1X4_2.54-SMD
- JP2: value (none) -> FIDUCIAL1X2; device pinhead (3):PINHD-1X6_2.54-SMD -> SparkFun:FIDUCIAL1X2
- JP3: value JUMPER-3PTH -> FIDUCIAL1X2; device SparkFun:JUMPER-3PTH -> SparkFun:FIDUCIAL1X2
- JP5: device pinhead (3):PINHD-1X4_2.54-SMD -> pinhead (3):PINHD-1X3_2.54-SMD
- JP6: value JUMPER-3PTH -> (none); device SparkFun:JUMPER-3PTH -> SparkFun:M031X03_NO_SILK
- JP7, JP9: value JUMPER-3PTH -> (none); device SparkFun:JUMPER-3PTH -> pinhead (3):PINHD-1X4_2.54-SMD
- LED1, LED4: device led:LEDCHIPLED_0805 -> led:LEDCHIP-LED0805
- Q1: value SUP90P06-09L -> ZXMN4A06; device transistor-power:IRF9530 -> ipc-7351-transistor:MOSFET-NCH_SOT-223
- Q3: value MOSFET-PCHANNELSMD -> AOT240L; device SparkFun:MOSFET-PCHANNELSMD -> transistor-power:IRF540
- R1: value ? -> (none)
- R10: value 22R -> 10K; device resistor:R-US_R0603 -> rcl:R-EU_R0603
- R11, R30: value 10k -> 10K; device resistor:R-US_R0603 -> rcl:R-EU_R0603
- R12: value 5.6K -> 10K; device resistor:R-US_R0603 -> rcl:R-EU_R0603
- R13: value 22R -> 5.6K
- R14: value 10k -> 22R
- R15: value 5.6K -> 10k
- R16: value (none) -> 10k; device rcl:R-EU_R0603 -> resistor:R-US_R0603
- R17: value (none) -> 1.5K
- R18, R4: value 10K -> (none)
- R19, R24, R26, R27: value 10K -> 1k
- R2: value 1k -> 5.6K; device rcl:R-EU_R0603 -> resistor:R-US_R0603
- R25, R28: value 2.2k -> 5k6
- R3: value (none) -> 1k
- R36: value 22R -> 5k6
- R39: value 2.2K -> 10K
- R41, R42: value 1k -> 2.2k
- R43: value 10k -> 5k6
- R45: value 10K -> 5k6
- R49: value 5.6K -> 10K
- R6: value 10K -> 22R; device rcl:R-EU_R0603 -> resistor:R-US_R0603
- R7: value 10K -> 10k; device rcl:R-EU_R0603 -> resistor:R-US_R0603
- R8: value 1k -> 10K
- X2: value MC2-G -> 5566-20; device con-phoenix-381_l:MC2-G -> con-molex:5566-20
- X3: value USB-MICROB -> MC2-G; device SparkFun:USB-MICROB -> con-phoenix-381_l:MC2-G
- X6: value MC2-G -> USB-MICROB; device con-phoenix-381_l:MC2-G -> SparkFun:USB-MICROB
- X7: value 5566-20 -> MC2-G; device con-molex:5566-20 -> con-phoenix-381_l:MC2-G
- renumbered C27 to C15, C28 to C16, C29 to C17, C30 to C18, C34 to C19, C35 to C20, IC14 to IC2, IC3 to IC1, JP21 to THERM., JP34 to LEDS, LED14 to VBB, LED16 to FAN, LED9 to USB, LPC2 to LPC1, M6 to M4, M7 to M3, Q12 to Q4, R65 to R9, R68 to R22, R74 to R34, R76 to R40, R90 to R23, RJ2 to RJ1, SJ6 to SJ1, X11 to X5, X9 to X1
Connections:
- net +12V: now also C11.2, C23.+, J4-2.S, R51.1, X2-10.S; no longer C4.2, C48.+, J1-2.S, R49.1, X7-10.S
- net +5V: now also J2-1.S, X2-19.S, X2-20.S, X2-4.S, X2-6.S; no longer J4-1.S, X7-19.S, X7-20.S, X7-4.S, X7-6.S
- net 3.3V: now also C7.2, C8.2, C9.+, D1.C, JP11.6, JP12.1, JP13.1, JP7.1, JP9.1, MS1.2, MS2.2, MS3.2, Q2.S, R10.2, R11.2, R12.2, R30.2, R31.2, R32.2, R33.2, R38.2, R39.2, R46.2, R47.2, R48.2, R49.2, R50.2, R8.2, X2-1.S, X2-11.S, X2-2.S; no longer C21.+, C24.2, C26.2, D2.C, JP1.2, JP12.2, JP13.2, JP17.1, JP18.1, JP2.6, JP3.1, JP5.1, Q3.S, R1.2, R18.2, R19.2, R2.2, R24.2, R26.2, R27.2, R4.2, R45.2, R57.2, R6.2, R61.2, R62.2, R66.2, R7.2, X7-1.S, X7-11.S, X7-2.S
- net 5V: now also JP13.3, JP7.3; no longer JP17.3, JP3.3
- net AVCC: now also AVCC.1
- net DIR3: now also JP16.3; no longer JP19.3
- net DIR4: now also M2.DIR; no longer M1.DIR
- net DIR5: now also M1.DIR; no longer M10.DIR
- net EN3: now also JP16.1; no longer JP19.1
- net EN4: now also M2./EN; no longer M1./EN
- net EN5: now also M1./EN; no longer M10./EN
- net GND: now also ATX.C, C10.-, C11.1, C13.1, C14.1, C22.2, C23.-, C25.-, C26.-, C4.-, C6.1, C7.1, C8.1, C9.-, D2.A, J2-2.S, JP10.5, JP11.1, JP12.2, JP14.2, JP16.4, JP5.1, JP8.5, LED1.C, LED2.C, LED3.C, M2.GND, M2.GND@1, PS_ON.2, Q1.S, Q3.S, R15.1, R16.1, R55.2, R7.2, RESET.3, RESET.4, X2-13.S, X2-15.S, X2-16.S, X2-17.S, X2-3.S, X2-5.S, X2-7.S, X4.2.SK, X6.GND, X7.1.SK, XMAX.2, XMIN.2, YMAX.2, YMIN.2, ZMAX.2, ZMIN.2; no longer C10.1, C11.-, C22.1, C23.1, C26.1, C4.1, C48.-, C6.-, C60.-, C61.-, C7.-, C8.2, C9.1, D3.A, J4-2.S, JP10.2, JP11.2, JP14.5, JP15.1, JP16.2, JP17.2, JP18.2, JP19.4, JP2.1, JP30.5, JP33.2, JP5.2, JP6.2, JP8.2, LED5.C, LED6.C, LED7.C, LED8.C, M10.GND, M10.GND@1, Q6.S, Q8.S, R11.1, R14.2, R30.1, R43.2, S4.3, S4.4, X2.2.SK, X3.GND, X4.1.SK, X7-13.S, X7-15.S, X7-16.S, X7-17.S, X7-3.S, X7-5.S, X7-7.S
- net ISP_BOOT: now also R31.1, S1.1, S1.2; no longer R24.1, S2.1, S2.2
- net LED1: now also R26.2; no longer R29.2
- net LED2: now also R29.2; no longer R41.2
- net LED3: now also R35.2; no longer R42.2
- net LED4: now also R37.2; no longer R44.2
- net MISO1: now also JP11.3; no longer JP2.3
- net MOSFET_DRIVE: now also C10.+, R13.1, X4.1.SK; no longer C60.+, R12.1, X2.1.SK
- net MOSI1: now also JP11.2; no longer JP2.2
- net MS0: now also M2.M0, MS3.1; no longer JP13.1, M10.M0
- net MS1: now also M2.M1, MS2.1; no longer JP12.1, M10.M1
- net MS2: now also M2.M2, MS1.1; no longer JP1.1, M10.M2
- net N$1: now also X6.D+; no longer X3.D+
- net N$10: now also LED1.A, R26.1; no longer LED5.A, R29.1
- net N$105: now also BIG.A, R13.2; no longer LED2.A, R12.2
- net N$107: now also R52.1; no longer R36.1
- net N$11: now also J3-3.S, M2.B1; no longer J6-3.S, M1.B1
- net N$12: now also Q2.D, R17.2; no longer Q3.D, R67.2
- net N$126: now also R54.1; no longer R39.1
- net N$128: now also R51.2; no longer R49.2
- net N$13: now also J3-4.S, M2.B2; no longer J6-4.S, M1.B2
- net N$135: now also D3.A, Q5.G, R55.1; no longer D4.A, Q1.G, R53.1
- net N$14: now also JP13.2, R19.2, R24.2, R27.2, R44.2, XMAX.3, XMIN.3, YMAX.3, YMIN.3, ZMAX.3, ZMIN.3; no longer JP10.3, JP11.3, JP3.2, JP6.3, JP7.3, JP8.3, JP9.3, R69.2, R70.2, R72.2, R78.2
- net N$140: now also C24.2; no longer C10.2
- net N$146: now also J1-3.S, M1.B1; no longer J5-3.S, M10.B1
- net N$147: now also J1-4.S, M1.B2; no longer J5-4.S, M10.B2
- net N$148: now also J1-2.S, M1.A1; no longer J5-2.S, M10.A1
- net N$149: now also J1-1.S, M1.A2; no longer J5-1.S, M10.A2
- net N$15: now also R43.1, ZMIN.1; no longer JP6.1, R77.1
- net N$152: now also M1./SLEEP, R11.1; no longer M10./SLEEP, R57.1
- net N$153: now also M1./RESET, R12.1; no longer M10./RESET, R62.1
- net N$16: now also R19.1, XMIN.1; no longer JP11.1, R69.1
- net N$17: now also R49.1; no longer R4.1
- net N$18: now also R24.1, R25.1, XMAX.1; no longer JP10.1, R70.1, R71.1
- net N$19: now also R27.1, R28.1, YMIN.1; no longer JP9.1, R72.1, R73.1
- net N$2: now also X6.D-; no longer X3.D-
- net N$20: now also R36.1, YMAX.1; no longer JP8.1, R75.1
- net N$21: now also J3-2.S, M2.A1; no longer J6-2.S, M1.A1
- net N$22: now also J5-3.S; no longer J3-3.S
- net N$23: now also JP7.4; no longer JP17.4
- net N$234234: now also JP15.1, PLAY.C, R33.1; no longer JP4.1, LED1.C, R2.1
- net N$24: now also R44.1, R45.1, ZMAX.1; no longer JP7.1, R78.1, R79.1
- net N$25: now also J5-4.S; no longer J3-4.S
- net N$26: now also J5-2.S; no longer J3-2.S
- net N$27: now also R41.2, R42.2; no longer R25.2, R28.2
- net N$28: now also J5-1.S; no longer J3-1.S
- net N$3: now also J6-3.S; no longer J2-3.S
- net N$30: now also R47.1; no longer R18.1
- net N$31: now also J3-1.S, M2.A2; no longer J6-1.S, M1.A2
- net N$32: now also M2./SLEEP, R38.1; no longer M1./SLEEP, R6.1
- net N$33: now also M2./RESET, R39.1; no longer M1./RESET, R7.1
- net N$34: now also C6.2, R3.2, X2-9.S; no longer C9.2, R8.2, X7-9.S
- net N$35: now also X2-8.S; no longer X7-8.S
- net N$36: now also ATX.A, R3.1; no longer LED4.A, R8.1
- net N$37: now also PS_ON.1, X2-14.S; no longer JP16.1, X7-14.S
- net N$38: now also JP5.2, R4.1; no longer JP15.2, R3.1
- net N$39: now also R1.2; no longer R16.2
- net N$4: now also J6-4.S; no longer J2-4.S
- net N$40: now also R14.1; no longer R10.1
- net N$41: now also R18.1; no longer R17.1
- net N$5: now also LED4.A, R37.1; no longer LED8.A, R44.1
- net N$6: now also LED3.A, R35.1; no longer LED7.A, R42.1
- net N$67: now also R50.1; no longer R26.1
- net N$68: now also R48.1; no longer R27.1
- net N$7: now also LED2.A, R29.1; no longer LED6.A, R41.1
- net N$74: now also Q1.G, R6.1; no longer Q8.G, R13.1
- net N$8: now also J6-2.S; no longer J2-2.S
- net N$81: now also R2.2, SMALL.A; no longer LED3.A, R15.2
- net N$88: now also Q1.D, SMALL.C, X3.2.SK; no longer LED3.C, Q8.D, X6.2.SK
- net N$9: now also J6-1.S; no longer J2-1.S
- net N$92: now also BIG.C, Q3.D; no longer LED2.C, Q6.D
- net N$96: now also J4-1.S; no longer J1-1.S
- net P1_22: now also C22.1, D1.A, D2.C, J2-3.S, JP10.1, R46.1; no longer C8.1, D2.A, D3.C, J4-3.S, JP14.1, R1.1
- net P1_23: now also JP10.2; no longer JP14.2
- net P1_30: now also JP10.4; no longer JP14.4
- net P1_31: now also JP10.3; no longer JP14.3
- net P2.6: now also JP8.1, R52.2, R53.1; no longer JP30.1, R36.2, R43.1
- net P2.7: now also JP8.4; no longer JP30.4
- net P2.9: now also Q2.G; no longer Q3.G
- net PLAY: now also JP14.1, R32.1, S2.1, S2.2; no longer JP33.1, R45.1, S4.1, S4.2
- net PLAY_LED: now also JP15.2, PLAY.A; no longer JP4.2, LED1.A
- net POT_SCL: now also JP9.4; no longer JP18.4
- net POT_SDA: now also JP9.3; no longer JP18.3
- net PWM0: now also JP8.2, R6.2, R7.1; no longer JP30.2, R13.2, R14.1
- net PWM1: now also JP8.3, R16.2; no longer JP30.3, R11.2
- net PWM1_FET: now also Q3.G, R14.2; no longer Q6.G, R10.2
- net RESET: now also R1.1, R30.1, RESET.1, RESET.2; no longer R16.1, R19.1, S1.1, S1.2
- net RX_0: now also R4.2; no longer R3.2
- net SCK1: now also JP11.4; no longer JP2.4
- net SCL: now also JP12.4, R41.1; no longer JP5.4, R25.1
- net SDA: now also JP12.3, R42.1; no longer JP5.3, R28.1
- net SD_CD: now also JP6.3; no longer JP20.3
- net SD_CS: now also R8.1; no longer R66.1
- net SD_IRQ: now also JP6.1; no longer JP20.1
- net SD_MOSI: now also R10.1; no longer R61.1
- net SD_WP: now also JP6.2; no longer JP20.2
- net SMALL_MOSFET_POWER: now also C1.+, R2.1, X3.1.SK; no longer C61.+, R15.1, X6.1.SK
- net SSDFGSDFG: now also R15.2; no longer R30.2
- net SSEL1: now also JP11.5; no longer JP2.5
- net STP3: now also JP16.2; no longer JP19.2
- net STP4: now also M2.STEP; no longer M1.STEP
- net STP5: now also M1.STEP; no longer M10.STEP
- net TH1: now also C2.+; no longer C5.+
- net TH2: now also C3.+; no longer C7.+
- net TH3: now also C4.+; no longer C11.+
- net TH4: now also C5.+; no longer C12.+
- net TX_0: now also JP5.3; no longer JP15.3
- net USB_D+: now also C14.2, R17.1; no longer C23.2, R67.1
- net USB_D-: now also C13.2; no longer C22.2
- net VBB: now also C12.+, C21.+, C25.+, C26.+, D3.C, M2.VMOT, Q5.S, R54.2; no longer C1.+, C2.+, C3.+, C6.+, D4.C, M10.VMOT, Q1.S, R39.2
- net VBB_IN: now also Q5.D, X7.2.SK; no longer Q1.D, X4.2.SK
- net VUSB: now also R18.2, X6.VBUS; no longer R17.2, X3.VBUS
- net X_MAX: now also R25.2; no longer R71.2
- net Y_MAX: now also R36.2; no longer R75.2
- net Y_MIN: now also R28.2; no longer R73.2
- net Z_MAX: now also R45.2; no longer R79.2
- net Z_MIN: now also R43.2; no longer R77.2
Other:
- note added: "AVCC connection to Xpresso!"
- note added: "Additional Stepper connector"
- moved on the sheet: C1, C12, C2, C21, C22, C24, C3, C5, C8, D2, J1-1, J1-2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
